Commit message: Updated files

File: robot_demo_description/urdf/robot_demo.urdf (robot description, URDF)
Before this commit: robot robot_demo, 5 links, 4 joints
Links:
- added link arm_base_link; visual box size=0.1 0.1 0.05
- added link arm_link_1, mass 1; collision box size=0.05 0.05 0.5; visual box size=0.05 0.05 0.5
- added link arm_link_2, mass 1; collision box size=0.05 0.05 0.5; visual box size=0.05 0.05 0.5
- added link dummy_link
Joints:
- added joint base_arm_base_joint: type revolute, parent base_link, child arm_base_link, origin xyz=0 0 0.1 rpy=0 0 0, axis 0 0 1, limit lower=-2.0944 upper=2.0944 effort=1000.0 velocity=0.5
- added joint base_joint: type fixed, parent dummy_link, child base_link, origin xyz=0.0 0.0 0.05 rpy=0.0 0.0 0.0
- added joint joint_arm1_arm2: type revolute, parent arm_link_1, child arm_link_2, origin xyz=0.05 0.0 0.3 rpy=0 0 0, axis 1 0 0, limit lower=-2.0944 upper=2.0944 effort=1000.0 velocity=0.5
- added joint joint_arm_base_arm_link_1: type revolute, parent arm_base_link, child arm_link_1, origin xyz=0 0 0.125 rpy=0 0 0, axis 1 0 0, limit lower=-1.57075 upper=1.57075 effort=1000.0 velocity=0.5
- joint base_wheel_2: origin xyz=0 0 0 rpy=0 0 0 -> xyz=-0.1 0.1 0.0 rpy=0 0 0
- joint base_wheel_3: origin xyz=0 0 0 rpy=0 0 0 -> xyz=0.1 -0.1 0.0 rpy=0 0 0
- joint base_wheel_4: origin xyz=0 0 0 rpy=0 0 0 -> xyz=-0.1 -0.1 0.0 rpy=0 0 0
